File: pcb/marco-keyboard.kicad_pcb (KiCad board)
At the start: 2 copper layers, 31 parts, among them J1 TYPE-C-31-M-12, J2 ICSP, SW0 CherryMX, SW1 CherryMX, SW2 CherryMX, SW3 CherryMX, SW4 CherryMX, SW5 CherryMX, SW6 CherryMX, U1 ATmega32U4-MUR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

Commit message: First version almost done
Parts:
- removed FB1, FB2: 50 @ 100MHz, Capacitor_SMD:C_0805_2012Metric
- added H1: MountingHole_Pad, MountingHole:MountingHole_2.2mm_M2_Pad, F.Cu at (125.1, 84.8)
- added H2: MountingHole_Pad, MountingHole:MountingHole_2.2mm_M2_Pad, F.Cu at (125.1, 58.1)
- added H3: MountingHole_Pad, MountingHole:MountingHole_2.2mm_M2_Pad, F.Cu at (174.1, 58.1)
- SW6: footprint Button_Switch_Keyboard:SW_Cherry_MX_2.00u_Vertical_PCB -> Custom:SW_Cherry_MX_2.00u_Vertical_PCB_unsupported
- moved R1 61.7 mm to (185.0, 57.4), turned to 180 degrees
- moved C2 37.3 mm to (177.6, 79.2), turned to 90 degrees
- moved C3 37.3 mm to (173.3, 83.5), turned to 180 degrees
- moved C7 31.8 mm to (183.4, 79.2), turned to 90 degrees
- moved F1 31.1 mm to (185.3, 79.2), turned to 90 degrees
- moved C1 28.4 mm to (186.7, 84.4)
- moved C5 27.0 mm to (173.3, 89.0), turned to 180 degrees
- moved C6 24.7 mm to (186.7, 82.8)
- moved C4 24.1 mm to (186.7, 87.4)
- moved J2 21.5 mm to (184.5, 61.1), turned to 0 degrees
- moved R4 20.2 mm to (186.7, 89.0)
- moved C8 15.1 mm to (166.3, 87.3), turned to 315 degrees
- moved U1 14.9 mm to (179.3, 85.6)
- moved C9 13.9 mm to (166.5, 83.3), turned to 45 degrees
- moved R3 12.8 mm to (181.4, 79.2)
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Connections:
- F1 pad 1: Net-(F1-Pad1) -> +5V
- J1 pad S1: Net-(FB2-Pad2) -> GND
- J1 pad S2: Net-(FB2-Pad2) -> GND
- J1 pad S3: Net-(FB2-Pad2) -> GND
- J1 pad S4: Net-(FB2-Pad2) -> GND
- U1 pad 18: BTN0 -> Net-(U1-Pad18)
- U1 pad 19: BTN1 -> BTN6
- U1 pad 20: BTN2 -> BTN4
- U1 pad 21: BTN3 -> BTN5
- U1 pad 22: BTN5 -> BTN2
- U1 pad 25: BTN4 -> BTN3
- U1 pad 26: BTN6 -> BTN0
- U1 pad 27: Net-(U1-Pad27) -> BTN1
Routing:
- net +5V: track 0.00 -> 243.6 mm, vias 0 -> 4
- net BTN0: track 0.00 -> 85.4 mm
- net BTN1: track 0.00 -> 68.7 mm
- net BTN2: track 0.00 -> 63.0 mm
- net BTN4: track 0.00 -> 48.4 mm
- net BTN3: track 0.00 -> 47.7 mm
- net RESET: track 0.00 -> 36.5 mm, vias 0 -> 1
- net GND: track 0.00 -> 35.8 mm, vias 0 -> 4
- net BTN6: track 0.00 -> 34.0 mm, vias 0 -> 1
- net Net-(R5-Pad1): track 0.00 -> 32.7 mm, vias 0 -> 2
- net BTN5: track 0.00 -> 29.9 mm
- net MOSI: track 0.00 -> 29.1 mm
- net MISO: track 0.00 -> 26.2 mm
- net SCLK: track 0.00 -> 25.3 mm, vias 0 -> 2
- net /VBUS: track 0.00 -> 17.1 mm
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- added copper zone on B.Cu, net GND
- added copper zone on F.Cu, net GND
Other:
- board outline added: 88.9 x 43.2 mm
- board text added: "Casteel"
- board text added: "ICSP"
- board text added: "JLCJLCJLCJLC"
- board text added: "Launchpad"
- board text added: "Martijn"
- board text added: "Rev 1.0"

Commit message: Created some files
Parts:
- added REF**: MountingHole_1.152mm, Custom:JLCPCB_Mountinghole_1.152mm, F.Cu at (189.9, 52.3)
- added REF**: MountingHole_1.152mm, Custom:JLCPCB_Mountinghole_1.152mm, F.Cu at (110.1, 85.7)
- added REF**: MountingHole_1.152mm, Custom:JLCPCB_Mountinghole_1.152mm, F.Cu at (110.1, 56.5)
Routing:
- net GND: track 35.8 -> 34.5 mm, vias 4 -> 3

Commit message: This looks like a good version
Parts:
- C1: value 100nf -> 0.1uf
