File: pcb/marco-keyboard.sch (KiCad schematic (older format))
At the start: 31 parts, among them J1 TYPE-C-31-M-12, J2 ICSP, SW0 CherryMX, SW1 CherryMX, SW2 CherryMX, SW3 CherryMX, SW4 CherryMX, SW5 CherryMX, SW6 CherryMX, U1 ATmega32U4-MUR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

Commit message: First version almost done
Parts:
- removed FB1, FB2: 50 @ 100MHz, Capacitor_SMD:C_0805_2012Metric, symbol Device:Ferrite_Bead_Small
- added H1, H2, H3: MountingHole_Pad, MountingHole:MountingHole_2.2mm_M2_Pad, symbol Mechanical:MountingHole_Pad
- SW6: footprint Button_Switch_Keyboard:SW_Cherry_MX_2.00u_Vertical_PCB -> Custom:SW_Cherry_MX_2.00u_Vertical_PCB_unsupported
Connections:
- net +5V: now also F1.1
- net BTN0: now also U1.26 (PD6); no longer U1.18 (PD0)
- net BTN1: now also U1.27 (PD7); no longer U1.19 (PD1)
- net BTN2: now also U1.22 (PD5); no longer U1.20 (PD2)
- net BTN3: now also U1.25 (PD4); no longer U1.21 (PD3)
- net BTN4: now also U1.20 (PD2); no longer U1.25 (PD4)
- net BTN5: now also U1.21 (PD3); no longer U1.22 (PD5)
- net BTN6: now also U1.19 (PD1); no longer U1.26 (PD6)
- net GND: now also J1.S1 (SHIELD), J1.S2 (SHIELD__1), J1.S3 (SHIELD__2), J1.S4 (SHIELD__3), H1.1, H2.1, H3.1
Changed lines of the file:
@@
 encoding utf-8
 Sheet 1 1
-Title "Macro-keyboard"
-Date "2021-03-14"
+Title "launchpad"
+Date "2021-03-21"
 Rev "1.0"
 Comp ""
@@
 Text GLabel 3350 3600 2    50   Input ~ 0
 MISO
-Text GLabel 3350 4500 2    50   Input ~ 0
+Text GLabel 3350 5100 2    50   Input ~ 0
 BTN0
+Text GLabel 3350 5200 2    50   Input ~ 0
+BTN1
+Text GLabel 3350 5000 2    50   Input ~ 0
+BTN2
+Text GLabel 3350 4900 2    50   Input ~ 0
+BTN3
+Text GLabel 3350 4700 2    50   Input ~ 0
+BTN4
+Text GLabel 3350 4800 2    50   Input ~ 0
+BTN5
 Text GLabel 3350 4600 2    50   Input ~ 0
-BTN1
-Text GLabel 3350 4700 2    50   Input ~ 0
-BTN2
-Text GLabel 3350 4800 2    50   Input ~ 0
-BTN3
-Text GLabel 3350 4900 2    50   Input ~ 0
-BTN4
-Text GLabel 3350 5000 2    50   Input ~ 0
-BTN5
-Text GLabel 3350 5100 2    50   Input ~ 0
 BTN6
 $Comp
@@
 NoConn ~ 3350 4300
 NoConn ~ 3350 5500
-NoConn ~ 3350 5200
+NoConn ~ 3350 4500
 NoConn ~ 3350 5800
 NoConn ~ 3350 5900
@@
 $EndComp
 $Comp
-L Device:Ferrite_Bead_Small FB2
-U 1 1 60513CFA
-P 9700 2700
-F 0 "FB2" V 9650 2850 50  0000 C CNN
-F 1 "50 @ 100MHz" V 9750 3000 50  0000 C CNN
-F 2 "Capacitor_SMD:C_0805_2012Metric" V 9630 2700 50  0001 C CNN
-F 3 "~" H 9700 2700 50  0001 C CNN
-F 4 "GZ2012D601TF" V 9700 2700 50  0001 C CNN "LCSC"
-	1    9700 2700
-	0    1    1    0
-$EndComp
-$Comp
 L Device:R_Small R7
 U 1 1 605178D0
@@
 Wire Wire Line
 	9950 2350 9950 2700
-Wire Wire Line
-	9800 2700 9950 2700
 Connection ~ 9950 2700
 Wire Wire Line
@@
 Wire Wire Line
 	9500 2650 9500 2700
-Wire Wire Line
-	9500 2700 9600 2700
 Connection ~ 9500 2700
 Wire Wire Line
@@
 $EndComp
 $Comp
-L Device:Ferrite_Bead_Small FB1
-U 1 1 6052AB28
-P 10000 1750
-F 0 "FB1" V 9950 1900 50  0000 C CNN
-F 1 "50 @ 100MHz" V 10050 2050 50  0000 C CNN
-F 2 "Capacitor_SMD:C_0805_2012Metric" V 9930 1750 50  0001 C CNN
-F 3 "~" H 10000 1750 50  0001 C CNN
-F 4 "GZ2012D601TF" V 10000 1750 50  0001 C CNN "LCSC"
-	1    10000 1750
-	0    1    1    0
-$EndComp
-$Comp
 L power:+5V #PWR0111
 U 1 1 6052C012
-P 10250 1500
-F 0 "#PWR0111" H 10250 1350 50  0001 C CNN
-F 1 "+5V" H 10265 1673 50  0000 C CNN
-F 2 "" H 10250 1500 50  0001 C CNN
-F 3 "" H 10250 1500 50  0001 C CNN
-	1    10250 1500
+P 9950 1500
+F 0 "#PWR0111" H 9950 1350 50  0001 C CNN
+F 1 "+5V" H 9965 1673 50  0000 C CNN
+F 2 "" H 9950 1500 50  0001 C CNN
+F 3 "" H 9950 1500 50  0001 C CNN
+	1    9950 1500
 	1    0    0    -1
 $EndComp
@@
 F 0 "SW6" V 9446 4952 50  0000 R CNN
 F 1 "CherryMX" V 9355 4952 50  0000 R CNN
-F 2 "Button_Switch_Keyboard:SW_Cherry_MX_2.00u_Vertical_PCB" H 9400 5025 50  0001 C CNN
+F 2 "Custom:SW_Cherry_MX_2.00u_Vertical_PCB_unsupported" H 9400 5025 50  0001 C CNN
 F 3 "" H 9400 5025 50  0001 C CNN
 	1    9400 5000
@@
 	2100 4100 2150 4100
 Wire Wire Line
-	10250 1500 10250 1750
-Wire Wire Line
-	10250 1750 10100 1750
-Wire Wire Line
-	9900 1750 9800 1750
+	9950 1500 9950 1750
+Wire Wire Line
+	9950 1750 9800 1750
 Wire Wire Line
 	9400 1750 9500 1750
@@
 	1    0    0    -1
 $EndComp
+Wire Wire Line
+	9500 2700 9950 2700
+$Comp
+L Mechanical:MountingHole_Pad H1
+U 1 1 6063F17D
+P 5750 7200
+F 0 "H1" H 5750 7400 50  0000 C CNN
+F 1 "MountingHole_Pad" H 5950 6850 50  0000 C CNN
+F 2 "MountingHole:MountingHole_2.2mm_M2_Pad" H 5750 7200 50  0001 C CNN
+F 3 "~" H 5750 7200 50  0001 C CNN
+	1    5750 7200
+	1    0    0    -1
+$EndComp
+$Comp
+L Mechanical:MountingHole_Pad H3
+U 1 1 6057C618
+P 6150 7200
+F 0 "H3" H 6100 7400 50  0000 L CNN
+F 1 "MountingHole_Pad" H 6250 7158 50  0001 L CNN
+F 2 "MountingHole:MountingHole_2.2mm_M2_Pad" H 6150 7200 50  0001 C CNN
+F 3 "~" H 6150 7200 50  0001 C CNN
+	1    6150 7200
+	1    0    0    -1
+$EndComp
+$Comp
+L Mechanical:MountingHole_Pad H2
+U 1 1 6063EEEC
+P 5950 7200
+F 0 "H2" H 5900 7400 50  0000 L CNN
+F 1 "MountingHole_Pad" H 6050 7158 50  0001 L CNN
+F 2 "MountingHole:MountingHole_2.2mm_M2_Pad" H 5950 7200 50  0001 C CNN
+F 3 "~" H 5950 7200 50  0001 C CNN
+	1    5950 7200
+	1    0    0    -1
+$EndComp
+Wire Wire Line
+	5750 7300 5750 7350
+Wire Wire Line
+	5750 7350 5950 7350
+Wire Wire Line
+	6150 7300 6150 7350
+Wire Wire Line
+	5950 7300 5950 7350
+Connection ~ 5950 7350
+$Comp
+L power:GND #PWR0109
+U 1 1 60590B9D
+P 5950 7400
+F 0 "#PWR0109" H 5950 7150 50  0001 C CNN
+F 1 "GND" H 6100 7350 50  0000 C CNN
+F 2 "" H 5950 7400 50  0001 C CNN
+F 3 "" H 5950 7400 50  0001 C CNN
+	1    5950 7400
+	1    0    0    -1
+$EndComp
+Wire Wire Line
+	5950 7350 6150 7350
+Wire Wire Line
+	5950 7350 5950 7400
 $EndSCHEMATC

Commit message: Created some files
Parts:
- removed H1, H2, H3: MountingHole_Pad, MountingHole:MountingHole_2.2mm_M2_Pad, symbol Mechanical:MountingHole_Pad
- C1, C3, C4, C5, C6: LCSC (none) -> C14663
- C2: LCSC (none) -> C28323
- C7: LCSC (none) -> C15850
- C8, C9: LCSC (none) -> C1804
- D2: LCSC (none) -> C2286
- F1: LCSC (none) -> C261937
- J1: LCSC (none) -> C165948
- R1, R4: LCSC (none) -> C25804
- R2, R3: LCSC (none) -> C23345
- R5: LCSC (none) -> C21190
- R6, R7: LCSC (none) -> C23186
- U1: LCSC (none) -> C45874; LCSC Part # (none) -> C45874
- Y1: LCSC (none) -> C13738
Changed lines of the file:
@@
 F 2 "Package_DFN_QFN:QFN-44-1EP_7x7mm_P0.5mm_EP5.2x5.2mm" H 2750 4800 50  0001 C CIN
 F 3 "http://ww1.microchip.com/downloads/en/DeviceDoc/Atmel-7766-8-bit-AVR-ATmega16U4-32U4_Datasheet.pdf" H 2750 4800 50  0001 C CNN
+F 4 "C45874" H 2750 4800 50  0001 C CNN "LCSC Part #"
+F 5 "C45874" H 2750 4800 50  0001 C CNN "LCSC"
 	1    2750 4800
 	1    0    0    -1
@@
 F 2 "Resistor_SMD:R_0603_1608Metric" H 1950 4300 50  0001 C CNN
 F 3 "~" H 1950 4300 50  0001 C CNN
+F 4 "C23345" H 1950 4300 50  0001 C CNN "LCSC"
 	1    1950 4300
 	0    1    1    0
@@
 F 2 "Resistor_SMD:R_0603_1608Metric" H 1950 4400 50  0001 C CNN
 F 3 "~" H 1950 4400 50  0001 C CNN
+F 4 "C23345" H 1950 4400 50  0001 C CNN "LCSC"
 	1    1950 4400
 	0    1    1    0
@@
 F 2 "Capacitor_SMD:C_0603_1608Metric" H 1950 4600 50  0001 C CNN
 F 3 "~" H 1950 4600 50  0001 C CNN
+F 4 "C28323" H 1950 4600 50  0001 C CNN "LCSC"
 	1    1950 4600
 	0    1    1    0
@@
 F 2 "Capacitor_SMD:C_0603_1608Metric" H 1950 3900 50  0001 C CNN
 F 3 "~" H 1950 3900 50  0001 C CNN
+F 4 "C14663" H 1950 3900 50  0001 C CNN "LCSC"
 	1    1950 3900
 	0    1    1    0
@@
 F 2 "Resistor_SMD:R_0603_1608Metric" H 3500 5400 50  0001 C CNN
 F 3 "~" H 3500 5400 50  0001 C CNN
+F 4 "C25804" H 3500 5400 50  0001 C CNN "LCSC"
 	1    3500 5400
 	0    -1   -1   0
@@
 F 2 "Resistor_SMD:R_0603_1608Metric" H 1950 3100 50  0001 C CNN
 F 3 "~" H 1950 3100 50  0001 C CNN
+F 4 "C25804" H 1950 3100 50  0001 C CNN "LCSC"
 	1    1950 3100
 	1    0    0    -1
@@
 F 2 "LED_SMD:LED_0603_1608Metric" V 3650 6100 50  0001 C CNN
 F 3 "~" V 3650 6100 50  0001 C CNN
+F 4 "C2286" H 3650 6100 50  0001 C CNN "LCSC"
 	1    3650 6100
 	0    -1   -1   0
@@
 F 2 "Resistor_SMD:R_0603_1608Metric" H 3650 5850 50  0001 C CNN
 F 3 "~" H 3650 5850 50  0001 C CNN
+F 4 "C21190" H 3650 5850 50  0001 C CNN "LCSC"
 	1    3650 5850
 	1    0    0    -1
@@
 F 2 "Resistor_SMD:R_0603_1608Metric" H 7550 2700 50  0001 C CNN
 F 3 "~" H 7550 2700 50  0001 C CNN
+F 4 "C23186" H 7550 2700 50  0001 C CNN "LCSC"
 	1    7550 2700
 	1    0    0    -1
@@
 F 2 "Resistor_SMD:R_0603_1608Metric" H 9700 2350 50  0001 C CNN
 F 3 "~" H 9700 2350 50  0001 C CNN
+F 4 "C23186" H 9700 2350 50  0001 C CNN "LCSC"
 	1    9700 2350
 	0    1    1    0
@@
 F 2 "Fuse:Fuse_0603_1608Metric" H 9700 1750 50  0001 C CNN
 F 3 "~" H 9700 1750 50  0001 C CNN
+F 4 "C261937" H 9700 1750 50  0001 C CNN "LCSC"
 	1    9700 1750
 	-1   0    0    1
@@
 F 2 "Capacitor_SMD:C_0603_1608Metric" H 1450 1550 50  0001 C CNN
 F 3 "~" H 1450 1550 50  0001 C CNN
+F 4 "C14663" H 1450 1550 50  0001 C CNN "LCSC"
 	1    1450 1550
 	1    0    0    -1
@@
 F 2 "Capacitor_SMD:C_0603_1608Metric" H 3050 1550 50  0001 C CNN
 F 3 "~" H 3050 1550 50  0001 C CNN
+F 4 "C15850" H 3050 1550 50  0001 C CNN "LCSC"
 	1    3050 1550
 	1    0    0    -1
@@
 F 2 "Capacitor_SMD:C_0603_1608Metric" H 1850 1550 50  0001 C CNN
 F 3 "~" H 1850 1550 50  0001 C CNN
+F 4 "C14663" H 1850 1550 50  0001 C CNN "LCSC"
 	1    1850 1550
 	1    0    0    -1
@@
 F 2 "Capacitor_SMD:C_0603_1608Metric" H 2650 1550 50  0001 C CNN
 F 3 "~" H 2650 1550 50  0001 C CNN
+F 4 "C14663" H 2650 1550 50  0001 C CNN "LCSC"
 	1    2650 1550
 	1    0    0    -1
@@
 F 2 "Capacitor_SMD:C_0603_1608Metric" H 2250 1550 50  0001 C CNN
 F 3 "~" H 2250 1550 50  0001 C CNN
+F 4 "C14663" H 2250 1550 50  0001 C CNN "LCSC"
 	1    2250 1550
 	1    0    0    -1
@@
 F 2 "Crystal:Crystal_SMD_3225-4Pin_3.2x2.5mm" H 5500 5750 50  0001 C CNN
 F 3 "~" H 5500 5750 50  0001 C CNN
+F 4 "C13738" H 5500 5750 50  0001 C CNN "LCSC"
 	1    5500 5750
 	1    0    0    -1
@@
 F 2 "Capacitor_SMD:C_0603_1608Metric" H 5150 6050 50  0001 C CNN
 F 3 "~" H 5150 6050 50  0001 C CNN
+F 4 "C1804" H 5150 6050 50  0001 C CNN "LCSC"
 	1    5150 6050
 	-1   0    0    1
@@
 F 2 "Capacitor_SMD:C_0603_1608Metric" H 5850 6050 50  0001 C CNN
 F 3 "~" H 5850 6050 50  0001 C CNN
+F 4 "C1804" H 5850 6050 50  0001 C CNN "LCSC"
 	1    5850 6050
 	-1   0    0    1
@@
 F 6 "Manufacturer Recommendations" H 8700 2150 50  0001 L BNN "STANDARD"
 F 7 "HRO Electronics" H 8700 2150 50  0001 L BNN "MANUFACTURER"
+F 8 "C165948" H 8700 2150 50  0001 C CNN "LCSC"
 	1    8700 2150
 	1    0    0    -1
@@
 Wire Wire Line
 	9500 2700 9950 2700
-$Comp
-L Mechanical:MountingHole_Pad H1
-U 1 1 6063F17D
-P 5750 7200
-F 0 "H1" H 5750 7400 50  0000 C CNN
-F 1 "MountingHole_Pad" H 5950 6850 50  0000 C CNN
-F 2 "MountingHole:MountingHole_2.2mm_M2_Pad" H 5750 7200 50  0001 C CNN
-F 3 "~" H 5750 7200 50  0001 C CNN
-	1    5750 7200
-	1    0    0    -1
-$EndComp
-$Comp
-L Mechanical:MountingHole_Pad H3
-U 1 1 6057C618
-P 6150 7200
-F 0 "H3" H 6100 7400 50  0000 L CNN
-F 1 "MountingHole_Pad" H 6250 7158 50  0001 L CNN
-F 2 "MountingHole:MountingHole_2.2mm_M2_Pad" H 6150 7200 50  0001 C CNN
-F 3 "~" H 6150 7200 50  0001 C CNN
-	1    6150 7200
-	1    0    0    -1
-$EndComp
-$Comp
-L Mechanical:MountingHole_Pad H2
-U 1 1 6063EEEC
-P 5950 7200
-F 0 "H2" H 5900 7400 50  0000 L CNN
-F 1 "MountingHole_Pad" H 6050 7158 50  0001 L CNN
-F 2 "MountingHole:MountingHole_2.2mm_M2_Pad" H 5950 7200 50  0001 C CNN
-F 3 "~" H 5950 7200 50  0001 C CNN
-	1    5950 7200
-	1    0    0    -1
-$EndComp
-Wire Wire Line
-	5750 7300 5750 7350
-Wire Wire Line
-	5750 7350 5950 7350
-Wire Wire Line
-	6150 7300 6150 7350
-Wire Wire Line
-	5950 7300 5950 7350
-Connection ~ 5950 7350
-$Comp
-L power:GND #PWR0109
-U 1 1 60590B9D
-P 5950 7400
-F 0 "#PWR0109" H 5950 7150 50  0001 C CNN
-F 1 "GND" H 6100 7350 50  0000 C CNN
-F 2 "" H 5950 7400 50  0001 C CNN
-F 3 "" H 5950 7400 50  0001 C CNN
-	1    5950 7400
-	1    0    0    -1
-$EndComp
-Wire Wire Line
-	5950 7350 6150 7350
-Wire Wire Line
-	5950 7350 5950 7400
 $EndSCHEMATC

Commit message: Fixed some things on the bom
Parts:
- C2: LCSC C28323 -> C15849
- R2, R3: LCSC C23345 -> C1653
Changed lines of the file:
@@
 F 2 "Resistor_SMD:R_0603_1608Metric" H 1950 4300 50  0001 C CNN
 F 3 "~" H 1950 4300 50  0001 C CNN
-F 4 "C23345" H 1950 4300 50  0001 C CNN "LCSC"
+F 4 "C1653" H 1950 4300 50  0001 C CNN "LCSC"
 	1    1950 4300
 	0    1    1    0
@@
 F 2 "Resistor_SMD:R_0603_1608Metric" H 1950 4400 50  0001 C CNN
 F 3 "~" H 1950 4400 50  0001 C CNN
-F 4 "C23345" H 1950 4400 50  0001 C CNN "LCSC"
+F 4 "C1653" H 1950 4400 50  0001 C CNN "LCSC"
 	1    1950 4400
 	0    1    1    0
@@
 F 2 "Capacitor_SMD:C_0603_1608Metric" H 1950 4600 50  0001 C CNN
 F 3 "~" H 1950 4600 50  0001 C CNN
-F 4 "C28323" H 1950 4600 50  0001 C CNN "LCSC"
+F 4 "C15849" H 1950 4600 50  0001 C CNN "LCSC"
 	1    1950 4600
 	0    1    1    0

Commit message: This looks like a good version
Parts:
- C1: value 100nf -> 0.1uf
- C7: LCSC C15850 -> C1634
- C8, C9: LCSC C1804 -> C1653
- R2, R3: LCSC C1653 -> C23345
Changed lines of the file:
@@
 F 2 "Resistor_SMD:R_0603_1608Metric" H 1950 4300 50  0001 C CNN
 F 3 "~" H 1950 4300 50  0001 C CNN
-F 4 "C1653" H 1950 4300 50  0001 C CNN "LCSC"
+F 4 "C23345" H 1950 4300 50  0001 C CNN "LCSC"
 	1    1950 4300
 	0    1    1    0
@@
 F 2 "Resistor_SMD:R_0603_1608Metric" H 1950 4400 50  0001 C CNN
 F 3 "~" H 1950 4400 50  0001 C CNN
-F 4 "C1653" H 1950 4400 50  0001 C CNN "LCSC"
+F 4 "C23345" H 1950 4400 50  0001 C CNN "LCSC"
 	1    1950 4400
 	0    1    1    0
@@
 F 4 "C15849" H 1950 4600 50  0001 C CNN "LCSC"
 	1    1950 4600
-	0    1    1    0
-$EndComp
-$Comp
-L Device:C_Small C1
-U 1 1 604F1B66
-P 1950 3900
-F 0 "C1" V 1900 3800 50  0000 C CNN
-F 1 "100nf" V 2000 3750 50  0000 C CNN
-F 2 "Capacitor_SMD:C_0603_1608Metric" H 1950 3900 50  0001 C CNN
-F 3 "~" H 1950 3900 50  0001 C CNN
-F 4 "C14663" H 1950 3900 50  0001 C CNN "LCSC"
-	1    1950 3900
 	0    1    1    0
 $EndComp
@@
 F 2 "Capacitor_SMD:C_0603_1608Metric" H 3050 1550 50  0001 C CNN
 F 3 "~" H 3050 1550 50  0001 C CNN
-F 4 "C15850" H 3050 1550 50  0001 C CNN "LCSC"
+F 4 "C1634" H 3050 1550 50  0001 C CNN "LCSC"
 	1    3050 1550
 	1    0    0    -1
@@
 F 2 "Capacitor_SMD:C_0603_1608Metric" H 5150 6050 50  0001 C CNN
 F 3 "~" H 5150 6050 50  0001 C CNN
-F 4 "C1804" H 5150 6050 50  0001 C CNN "LCSC"
+F 4 "C1653" H 5150 6050 50  0001 C CNN "LCSC"
 	1    5150 6050
 	-1   0    0    1
@@
 F 2 "Capacitor_SMD:C_0603_1608Metric" H 5850 6050 50  0001 C CNN
 F 3 "~" H 5850 6050 50  0001 C CNN
-F 4 "C1804" H 5850 6050 50  0001 C CNN "LCSC"
+F 4 "C1653" H 5850 6050 50  0001 C CNN "LCSC"
 	1    5850 6050
 	-1   0    0    1
@@
 Wire Wire Line
 	9500 2700 9950 2700
+$Comp
+L Device:C_Small C1
+U 1 1 604F1B66
+P 1950 3900
+F 0 "C1" V 1900 3800 50  0000 C CNN
+F 1 "0.1uf" V 2000 3750 50  0000 C CNN
+F 2 "Capacitor_SMD:C_0603_1608Metric" H 1950 3900 50  0001 C CNN
+F 3 "~" H 1950 3900 50  0001 C CNN
+F 4 "C14663" H 1950 3900 50  0001 C CNN "LCSC"
+	1    1950 3900
+	0    1    1    0
+$EndComp
 $EndSCHEMATC
